File: 040-05x-v2/040-05x-v2.kicad_pcb (KiCad board)
At the start: 2 copper layers, 21.8 x 21.3 mm, 6 parts, among them J2 Conn_01x12, J3 Conn_01x12, J4 USB_C_Receptacle_USB2.0_16P

Commit message: Add my own logo
Other:
- board text added: "acolombo"
- board text removed: "CasuaCoders.dev"
- board text removed: "JDS-040/05x V2"
Changed lines of the file:
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@@
 				(font
 					(size 1.27 1.27)
+					(thickness 0.15)
 				)
 			)
@@
 				(font
 					(size 1.27 1.27)
+					(thickness 0.15)
 				)
 			)
@@
 				(font
 					(size 1.27 1.27)
+					(thickness 0.15)
 				)
 			)
@@
 				(font
 					(size 1.27 1.27)
+					(thickness 0.15)
 				)
 			)
@@
 				(font
 					(size 1.27 1.27)
+					(thickness 0.15)
 				)
 			)
@@
 				(font
 					(size 1.27 1.27)
+					(thickness 0.15)
 				)
 			)
@@
 				(font
 					(size 1.27 1.27)
+					(thickness 0.15)
 				)
 			)
@@
 				(font
 					(size 1.27 1.27)
+					(thickness 0.15)
 				)
 			)
@@
 				(font
 					(size 1.27 1.27)
+					(thickness 0.15)
 				)
 			)
@@
 				(font
 					(size 1.27 1.27)
+					(thickness 0.15)
 				)
 			)
@@
 				(font
 					(size 1.27 1.27)
+					(thickness 0.15)
 				)
 			)
@@
 				(font
 					(size 1.27 1.27)
+					(thickness 0.15)
 				)
 			)
@@
 				(font
 					(size 1.27 1.27)
+					(thickness 0.15)
 				)
 			)
@@
 				(font
 					(size 1.27 1.27)
+					(thickness 0.15)
 				)
 			)
@@
 				(font
 					(size 1.27 1.27)
+					(thickness 0.15)
 				)
 			)
@@
 				(font
 					(size 1.27 1.27)
+					(thickness 0.15)
 				)
 			)
@@
 				(font
 					(size 1.27 1.27)
+					(thickness 0.15)
 				)
 			)
@@
 				(font
 					(size 1.27 1.27)
+					(thickness 0.15)
 				)
 			)
@@
 	)
 	(gr_line
+		(start 67.056 62.260521)
+		(end 67.056 63.239479)
+		(stroke
+			(width 0.14)
+			(type solid)
+			(color 255 0 0 1)
+		)
+		(layer "F.Mask")
+	)
+	(gr_line
+		(start 65.936813 63.998172)
+		(end 68.175188 63.998172)
+		(stroke
+			(width 0.14)
+			(type solid)
+			(color 255 0 0 1)
+		)
+		(layer "F.Mask")
+	)
+	(gr_line
+		(start 68.175188 63.034427)
+		(end 68.175188 63.998172)
+		(stroke
+			(width 0.14)
+			(type solid)
+			(color 255 0 0 1)
+		)
+		(layer "F.Mask")
+	)
+	(gr_poly
+		(pts
+			(xy 69.027146 63.592963) (xy 69.027146 64.590177) (xy 67.056 63.247417) (xy 65.084854 64.590177)
+			(xy 65.084854 63.592963) (xy 67.056 62.250467)
+		)
+		(stroke
+			(width 0.14)
+			(type solid)
+			(color 255 0 0 1)
+		)
+		(fill none)
+		(layer "F.Mask")
+	)
+	(gr_line
+		(start 65.936813 63.034427)
+		(end 65.936813 63.998172)
+		(stroke
+			(width 0.14)
+			(type solid)
+			(color 255 0 0 1)
+		)
+		(layer "F.Mask")
+	)
+	(gr_line
 		(start 62.738 67.056)
 		(end 62.738 78.74)
@@
 	)
 	(gr_line
-		(start 62.681 78.911226)
+		(start 62.681 78.5)
 		(end 62.681 66.911226)
 		(stroke
@@
 	(gr_line
 		(start 73.425561 57.404)
-		(end 73.425561 42.904)
-		(stroke
-			(width 0.25)
-			(type solid)
-		)
-		(layer "User.9")
-	)
-	(gr_line
-		(start 73.425561 57.404)
 		(end 58.925561 57.404)
 		(stroke
@@
 	)
 	(gr_line
-		(start 73.425561 57.404)
-		(end 73.425561 49.404)
-		(stroke
-			(width 0.25)
-			(type solid)
-		)
-		(layer "User.9")
-	)
-	(gr_line
 		(start 56.182605 58.618987)
 		(end 59.681 66.911226)
@@
 		(layer "User.9")
 	)
-	(gr_text "CasuaCoders.dev"
-		(at 64.262 78.486 90)
+	(gr_text "acolombo"
+		(at 67.056 68.5 0)
 		(layer "F.SilkS")
 		(effects
 			(font
-				(size 1 1)
-				(thickness 0.15)
+				(size 0.9 0.9)
+				(bold yes)
 			)
-			(justify left bottom)
-		)
-	)
-	(gr_text "JDS-040/05x V2"
-		(at 71.12 78.232 90)
-		(layer "F.SilkS")
-		(effects
-			(font
-				(size 1 1)
-				(thickness 0.15)
-			)
-			(justify left bottom)
+			(justify bottom)
 		)
 	)
@@
 		)
 	)
+	(group ""
+		(members "210dc0bd-ae2d-4272-874b-c80826d479df" "67dcd032-c3e2-4d1c-a284-9c6e37334f09"
+			"6ab9c270-8278-4edc-9b39-024ed65bed96" "77310da3-8e3c-4b53-be2a-a59240492e13"
+			"f3cf8eee-4b30-4c14-a99b-b7c3b473be58"
+		)
+	)
